File: eagle files/board design.brd (EAGLE design)
At the start: 168.9 x 116.5 mm, 35 parts

Commit message: 10/2/19
Parts:
- removed U$1, U$2: DC-DC-LM2596-DISP, uln2003:DC-DC-LM2596-DISP
- added C3, C4: (no value), rcl:E2,5-7
- added IC1: 7805T, linear:TO220H
- moved PCT1 75.1 mm to (67.9, 19.7), turned to 270 degrees
- moved U$3 66.1 mm to (14.6, 22.2), turned to 270 degrees
- moved PCT2 59.6 mm to (67.9, 36.2), turned to 270 degrees
- moved R2 56.5 mm to (61.6, 19.7)
- moved 2A4981-8 55.4 mm to (78.1, 28.6)
- moved BIPOLAR_2 55.4 mm to (102.2, 28.6)
- moved 2A498,9-16 55.4 mm to (90.8, 28.6)
- moved R1 55.4 mm to (16.5, 47.6)
- moved LIDAR 54.3 mm to (6.99, 52.7)
- moved 12V_INPUT 53.8 mm to (109.9, 43.8)
- moved C1 53.4 mm to (97.2, 45.1)
- moved 1A498-1-8 52.7 mm to (78.1, 62.9)
- moved BIPOLAR_1 52.7 mm to (102.2, 62.9)
- moved 1A498,9-16 52.7 mm to (90.8, 62.9)
- moved ZENER1 51.2 mm to (28.6, 55.2)
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Connections:
- new net N$37: C3.+, IC1.3, LIDAR.3, ZENER1.1
- net 5V: now also C4.+, IC1.1; no longer LIDAR.4, ZENER1.1
- net GND: now also C3.-, C4.-, IC1.2, LIDAR.4; no longer LIDAR.3
- net N$22: no longer U$2.OUT-
- net N$25: no longer U$2.OUT+
Routing:
- net N$37: track 0.00 -> 63.1 mm
- net N$4: track 62.8 -> 25.7 mm
- net 5V: track 238.5 -> 266.8 mm
- net N$32: track 42.6 -> 15.2 mm
- net N$18: track 38.7 -> 12.0 mm
- net N$3: track 57.7 -> 31.9 mm
- net N$33: track 48.7 -> 27.4 mm
- net N$25: track 52.6 -> 72.9 mm
- net N$8: track 20.8 -> 41.1 mm
- net N$28: track 17.7 -> 36.2 mm
- net N$2: track 55.7 -> 38.1 mm
- net N$26: track 15.6 -> 33.0 mm
- net N$27: track 16.7 -> 32.6 mm
- net N$17: track 6.53 -> 22.4 mm
- net N$20: track 29.5 -> 44.1 mm
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Other:
- board size 168.9 x 116.5 mm -> 115.6 x 89.5 mm
- board text added: "SHUBHAM R PANCHAL"

Commit message: 10/2/19 -2
Parts:
- moved PCT2 7.69 mm to (72.7, 42.2)
- moved PCT1 5.97 mm to (70.5, 25.1), turned to 90 degrees
- moved R3 5.46 mm to (53.3, 16.5)
- moved R4 4.72 mm to (58.7, 16.5)
- moved R2 4.27 mm to (64.5, 16.5)
- moved PCT3 3.98 mm to (71.1, 57.5)
- flipped 2A4981-8 to the bottom
Routing:
- net N$1: track 42.4 -> 0.00 mm
- net N$22: track 62.6 -> 97.1 mm
- net 5V: track 266.8 -> 293.2 mm
- net GND: track 279.8 -> 298.0 mm
- net N$8: track 41.1 -> 24.4 mm
- net N$24: track 12.1 -> 2.54 mm
- net N$33: track 27.4 -> 36.7 mm
- net N$17: track 22.4 -> 13.7 mm
- net N$23: track 10.2 -> 2.54 mm
- net N$32: track 15.2 -> 7.94 mm
- net N$31: track 26.3 -> 20.9 mm
- net N$18: track 12.0 -> 16.9 mm
- net N$2: track 38.1 -> 33.6 mm
- net N$6: track 12.0 -> 7.77 mm
- net N$19: track 18.9 -> 14.7 mm
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
Commit message: 12/2/19
Parts:
- removed JP8, JP9: (no value), pinhead:1X02
- removed U$3: DRIVER-ULN2003#MC, uln2003:DRIVER-ULN2003#MC
- added 5V_INPUT1, 5V_INPUT2: (no value), pinhead:1X02
- added JP1, JP2, JP3, JP4: (no value), pinhead:1X01
- added JP5, JP6: (no value), pinhead:1X07
- moved LED1 20.0 mm to (47.9, 4.13), turned to 270 degrees
- moved R4 12.4 mm to (46.4, 16.5)
- moved SERVO1 5.09 mm to (32.4, 13.0)
- moved SERVO2 5.09 mm to (32.4, 7.94)
- moved SERVO3 5.09 mm to (32.4, 2.86)
- moved C5 3.43 mm to (31.1, 29.8), turned to 180 degrees
- moved C1 3.27 mm to (100.0, 43.5), turned to 270 degrees
- moved R3 2.88 mm to (56.2, 16.2)
- moved C6 2.56 mm to (59.1, 78.4), turned to 90 degrees
- moved LED2 1.62 mm to (58.1, 4.13), turned to 270 degrees
- moved PCT2 1.31 mm to (72.4, 43.5)
- moved ZENER1 1.27 mm to (28.6, 56.5)
- moved R1 0.71 mm to (15.9, 47.3)
- moved C3 0.64 mm to (41.3, 77.5), turned to 90 degrees
- moved C4 0.45 mm to (31.4, 77.8), turned to 270 degrees
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Connections:
- removed net GND: C3.-, C4.-, C5.-, C6.-, C7.-, IC1.2, JP9.1, LED1.K, LED2.K, LIDAR.4, NANO1-15.4, NANO16-30.14, SERVO1.1, SERVO2.1, SERVO3.1, SP1.+, U$3.J3.1, ZENER1.2
- new net N$36: C5.-, C6.-, C7.-, JP2.1, LED1.K, LED2.K, SERVO1.1, SERVO2.1, SERVO3.1, SP1.+
- new net N$38: 5V_INPUT1.1, 5V_INPUT2.1, C3.-, C4.-, IC1.2, LIDAR.4, NANO1-15.4, NANO16-30.14, ZENER1.2
- net 5V: now also 5V_INPUT1.2, JP1.1; no longer JP9.2, NANO16-30.12, U$3.J3.2
- net GUC: now also JP4.1; no longer JP8.2
- net N$1: now also JP5.4; no longer U$3.J1.4
- net N$2: now also JP5.3; no longer U$3.J1.3
- net N$3: now also JP5.2; no longer U$3.J1.2
- net N$37: now also 5V_INPUT2.2, NANO16-30.12
- net N$4: now also JP5.1; no longer U$3.J1.1
- net VUC: now also JP3.1; no longer JP8.1
Routing:
- net N$36: track 0.00 -> 309.1 mm
- net GND: track 298.0 -> 0.00 mm
- net N$38: track 0.00 -> 140.4 mm
- net N$37: track 66.3 -> 140.9 mm
- net N$1: track 0.00 -> 38.8 mm
- net 5V: track 293.2 -> 304.1 mm
- net VUC: track 54.6 -> 63.1 mm
- net N$17: track 13.7 -> 6.69 mm
- net N$26: track 30.6 -> 36.9 mm
- net N$18: track 16.9 -> 10.8 mm
- net N$22: track 97.1 -> 103.2 mm
- net N$27: track 33.6 -> 39.5 mm
- net N$28: track 36.7 -> 42.2 mm
- net N$33: track 36.7 -> 34.4 mm
- net GUC: track 48.4 -> 46.5 mm
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- added copper zone on layer 16, net N$39
Other:
- board size 115.6 x 89.5 mm -> 24.1 x 44.1 mm

Commit message: first backup 15-2-18
Parts:
- removed 12V_INPUT, 5V_INPUT1: (no value), pinhead:1X02
- added JP10, JP7, JP8, JP9: (no value), pinhead:1X01
- renumbered IC1 to LM7805
Connections:
- net 5V: now also JP7.1; no longer 5V_INPUT1.2
- net N$22: now also JP10.1; no longer 12V_INPUT.2
- net N$25: now also JP9.1; no longer 12V_INPUT.1
- net N$38: now also JP8.1; no longer 5V_INPUT1.1
Routing:
- net N$38: track 140.4 -> 135.4 mm
- net N$22: track 103.2 -> 105.1 mm
Other:
- board outline removed
