File: eagle files/board design.sch (EAGLE design)
At the start: 35 parts

Commit message: 10/2/19
Parts:
- removed U$1, U$2: DC-DC-LM2596-DISP, uln2003:DC-DC-LM2596-DISP
- added C3, C4: (no value), rcl:CPOL-USE2.5-7
- added IC1: 7805T, linear:7805T
Connections:
- new net N$37: C3.+, IC1.VO, LIDAR.3, ZENER1.1
- net 5V: now also C4.+, IC1.VI; no longer LIDAR.4, ZENER1.1
- net GND: now also C3.-, C4.-, IC1.GND, LIDAR.4; no longer LIDAR.3
- net N$22: no longer U$2.OUT-
- net N$25: no longer U$2.OUT+
Other:
- moved on the sheet: ZENER1

Commit message: 12/2/19
Parts:
- removed JP8, JP9: (no value), pinhead:PINHD-1X2
- removed U$3: DRIVER-ULN2003#MC, uln2003:DRIVER-ULN2003#MC
- added 5V_INPUT1, 5V_INPUT2: (no value), pinhead:PINHD-1X2
- added JP1, JP2, JP3, JP4: (no value), pinhead:PINHD-1X1
- added JP5, JP6: (no value), pinhead:PINHD-1X7
Connections:
- removed net GND: C3.-, C4.-, C5.-, C6.-, C7.-, IC1.GND, JP9.1, LED1.C, LED2.C, LIDAR.4, NANO1-15.4, NANO16-30.14, SERVO1.1, SERVO2.1, SERVO3.1, SP1.2, U$3.GND, ZENER1.2
- new net N$36: C5.-, C6.-, C7.-, JP2.1, LED1.C, LED2.C, SERVO1.1, SERVO2.1, SERVO3.1, SP1.2
- new net N$38: 5V_INPUT1.1, 5V_INPUT2.1, C3.-, C4.-, IC1.GND, LIDAR.4, NANO1-15.4, NANO16-30.14, ZENER1.2
- net 5V: now also 5V_INPUT1.2, JP1.1; no longer JP9.2, NANO16-30.12, U$3.VCC.1
- net GUC: now also JP4.1; no longer JP8.2
- net N$1: now also JP5.4; no longer U$3.IN.4
- net N$2: now also JP5.3; no longer U$3.IN.3
- net N$3: now also JP5.2; no longer U$3.IN.2
- net N$37: now also 5V_INPUT2.2, NANO16-30.12
- net N$4: now also JP5.1; no longer U$3.IN.1
- net VUC: now also JP3.1; no longer JP8.1

Commit message: first backup 15-2-18
Parts:
- removed 12V_INPUT, 5V_INPUT1: (no value), pinhead:PINHD-1X2
- added JP10, JP7, JP8, JP9: (no value), pinhead:PINHD-1X1
- renumbered IC1 to LM7805
Connections:
- net 5V: now also JP7.1; no longer 5V_INPUT1.2
- net N$22: now also JP10.1; no longer 12V_INPUT.2
- net N$25: now also JP9.1; no longer 12V_INPUT.1
- net N$38: now also JP8.1; no longer 5V_INPUT1.1
Changed lines of the file:
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@@
 <part name="C6" library="rcl" deviceset="CPOL-US" device="E2.5-7"/>
 <part name="C7" library="rcl" deviceset="CPOL-US" device="E2.5-7"/>
-<part name="12V_INPUT" library="pinhead" deviceset="PINHD-1X2" device=""/>
 <part name="LIDAR" library="pinhead" deviceset="PINHD-1X4" device=""/>
 <part name="PCT3" library="resistor" deviceset="R-US_" device="0207/10"/>
@@
 <part name="PCT2" library="resistor" deviceset="R-US_" device="0207/10"/>
 <part name="ZENER1" library="resistor" deviceset="R-US_" device="0207/10"/>
-<part name="IC1" library="linear" deviceset="78*" device="T" technology="05"/>
+<part name="LM7805" library="linear" deviceset="78*" device="T" technology="05"/>
 <part name="C3" library="rcl" deviceset="CPOL-US" device="E2.5-7"/>
 <part name="C4" library="rcl" deviceset="CPOL-US" device="E2.5-7"/>
-<part name="5V_INPUT1" library="pinhead" deviceset="PINHD-1X2" device=""/>
 <part name="JP1" library="pinhead" deviceset="PINHD-1X1" device=""/>
 <part name="JP2" library="pinhead" deviceset="PINHD-1X1" device=""/>
@@
 <part name="JP5" library="pinhead" deviceset="PINHD-1X7" device=""/>
 <part name="JP6" library="pinhead" deviceset="PINHD-1X7" device=""/>
+<part name="JP7" library="pinhead" deviceset="PINHD-1X1" device=""/>
+<part name="JP8" library="pinhead" deviceset="PINHD-1X1" device=""/>
+<part name="JP9" library="pinhead" deviceset="PINHD-1X1" device=""/>
+<part name="JP10" library="pinhead" deviceset="PINHD-1X1" device=""/>
 </parts>
 <sheets>
@@
 <instance part="C6" gate="G$1" x="-5.08" y="7.62" rot="R270"/>
 <instance part="C7" gate="G$1" x="-5.08" y="-10.16" rot="R270"/>
-<instance part="12V_INPUT" gate="G$1" x="256.54" y="91.44"/>
 <instance part="LIDAR" gate="A" x="-2.54" y="78.74" rot="R180"/>
 <instance part="PCT3" gate="G$1" x="152.4" y="96.52" rot="R180"/>
@@
 <instance part="PCT2" gate="G$1" x="132.08" y="63.5" rot="R180"/>
 <instance part="ZENER1" gate="G$1" x="5.08" y="101.6" rot="R270"/>
-<instance part="IC1" gate="A1" x="-25.4" y="104.14"/>
+<instance part="LM7805" gate="A1" x="-25.4" y="104.14"/>
 <instance part="C3" gate="G$1" x="-10.16" y="101.6"/>
 <instance part="C4" gate="G$1" x="-40.64" y="101.6"/>
-<instance part="5V_INPUT1" gate="G$1" x="-63.5" y="101.6" rot="R180"/>
 <instance part="JP1" gate="G$1" x="271.78" y="68.58" rot="R180"/>
 <instance part="JP2" gate="G$1" x="271.78" y="60.96" rot="R180"/>
@@
 <instance part="JP5" gate="A" x="-40.64" y="63.5" rot="R180"/>
 <instance part="JP6" gate="A" x="-96.52" y="63.5" rot="R180"/>
+<instance part="JP7" gate="G$1" x="-86.36" y="101.6" rot="R180"/>
+<instance part="JP8" gate="G$1" x="-86.36" y="93.98" rot="R180"/>
+<instance part="JP9" gate="G$1" x="271.78" y="93.98"/>
+<instance part="JP10" gate="G$1" x="271.78" y="86.36"/>
 </instances>
 <busses>
@@
 <wire x1="233.68" y1="88.9" x2="241.3" y2="88.9" width="0.1524" layer="91"/>
 <wire x1="241.3" y1="88.9" x2="241.3" y2="91.44" width="0.1524" layer="91"/>
-<pinref part="12V_INPUT" gate="G$1" pin="2"/>
 <wire x1="241.3" y1="91.44" x2="254" y2="91.44" width="0.1524" layer="91"/>
 <wire x1="213.36" y1="116.84" x2="233.68" y2="116.84" width="0.1524" layer="91"/>
 <wire x1="233.68" y1="116.84" x2="233.68" y2="88.9" width="0.1524" layer="91"/>
+<pinref part="JP10" gate="G$1" pin="1"/>
+<wire x1="269.24" y1="86.36" x2="254" y2="86.36" width="0.1524" layer="91"/>
+<wire x1="254" y1="86.36" x2="254" y2="91.44" width="0.1524" layer="91"/>
 </segment>
 </net>
@@
 <wire x1="200.66" y1="119.38" x2="241.3" y2="119.38" width="0.1524" layer="91"/>
 <wire x1="241.3" y1="119.38" x2="241.3" y2="99.06" width="0.1524" layer="91"/>
-<pinref part="12V_INPUT" gate="G$1" pin="1"/>
 <wire x1="241.3" y1="99.06" x2="241.3" y2="93.98" width="0.1524" layer="91"/>
-<wire x1="241.3" y1="93.98" x2="254" y2="93.98" width="0.1524" layer="91"/>
 <wire x1="231.14" y1="99.06" x2="241.3" y2="99.06" width="0.1524" layer="91"/>
+<pinref part="JP9" gate="G$1" pin="1"/>
+<wire x1="269.24" y1="93.98" x2="241.3" y2="93.98" width="0.1524" layer="91"/>
 </segment>
 </net>
@@
 </segment>
 <segment>
-<pinref part="IC1" gate="A1" pin="VI"/>
+<pinref part="LM7805" gate="A1" pin="VI"/>
 <pinref part="C4" gate="G$1" pin="+"/>
 <wire x1="-35.56" y1="104.14" x2="-40.64" y2="104.14" width="0.1524" layer="91"/>
-<pinref part="5V_INPUT1" gate="G$1" pin="2"/>
-<wire x1="-60.96" y1="101.6" x2="-48.26" y2="101.6" width="0.1524" layer="91"/>
 <wire x1="-48.26" y1="101.6" x2="-48.26" y2="104.14" width="0.1524" layer="91"/>
 <wire x1="-48.26" y1="104.14" x2="-40.64" y2="104.14" width="0.1524" layer="91"/>
@@
 <wire x1="109.22" y1="114.3" x2="-73.66" y2="114.3" width="0.1524" layer="91"/>
 <wire x1="-73.66" y1="114.3" x2="-73.66" y2="101.6" width="0.1524" layer="91"/>
-<wire x1="-73.66" y1="101.6" x2="-60.96" y2="101.6" width="0.1524" layer="91"/>
+<wire x1="-73.66" y1="101.6" x2="-48.26" y2="101.6" width="0.1524" layer="91"/>
 <pinref part="JP1" gate="G$1" pin="1"/>
 <junction x="274.32" y="68.58"/>
+<pinref part="JP7" gate="G$1" pin="1"/>
+<wire x1="-83.82" y1="101.6" x2="-73.66" y2="101.6" width="0.1524" layer="91"/>
 </segment>
 </net>
@@
 <net name="N$37" class="0">
 <segment>
-<pinref part="IC1" gate="A1" pin="VO"/>
+<pinref part="LM7805" gate="A1" pin="VO"/>
 <pinref part="C3" gate="G$1" pin="+"/>
 <wire x1="-15.24" y1="104.14" x2="-10.16" y2="104.14" width="0.1524" layer="91"/>
@@
 <segment>
 <pinref part="C4" gate="G$1" pin="-"/>
-<pinref part="5V_INPUT1" gate="G$1" pin="1"/>
-<wire x1="-60.96" y1="99.06" x2="-48.26" y2="99.06" width="0.1524" layer="91"/>
 <wire x1="-48.26" y1="99.06" x2="-48.26" y2="96.52" width="0.1524" layer="91"/>
 <wire x1="-48.26" y1="96.52" x2="-40.64" y2="96.52" width="0.1524" layer="91"/>
-<pinref part="IC1" gate="A1" pin="GND"/>
+<pinref part="LM7805" gate="A1" pin="GND"/>
 <wire x1="-25.4" y1="96.52" x2="-40.64" y2="96.52" width="0.1524" layer="91"/>
 <pinref part="NANO1-15" gate="A" pin="4"/>
@@
 <pinref part="5V_INPUT2" gate="G$1" pin="1"/>
 <wire x1="-38.1" y1="78.74" x2="-25.4" y2="78.74" width="0.1524" layer="91"/>
-</segment>
-</net>
+<pinref part="JP8" gate="G$1" pin="1"/>
+<wire x1="-83.82" y1="93.98" x2="-76.2" y2="93.98" width="0.1524" layer="91"/>
+<wire x1="-76.2" y1="93.98" x2="-76.2" y2="99.06" width="0.1524" layer="91"/>
+<wire x1="-76.2" y1="99.06" x2="-48.26" y2="99.06" width="0.1524" layer="91"/>
+</segment>
+</net>
